File: BravaController/BravaController.kicad_sch (KiCad schematic)
At the start: 4 parts, among them U1 RASPBERRY_PI_ZERO_2_W, U2 74AHCT125

Commit message: Developed Draft Schematic for Design
Parts:
- added C1, C2: 10u, Capacitor_SMD:C_0805_2012Metric_Pad1.18x1.45mm_HandSolder, symbol Device:C
- added C3: 100n, Capacitor_SMD:C_0805_2012Metric_Pad1.18x1.45mm_HandSolder, symbol Device:C
- added C4: 150n, Capacitor_SMD:C_0805_2012Metric_Pad1.18x1.45mm_HandSolder, symbol Device:C
- added C5: 10n, Capacitor_SMD:C_0805_2012Metric_Pad1.18x1.45mm_HandSolder, symbol Device:C
- added D1, D10, D2, D5, D6, D7, D8, D9: LED, LED_SMD:LED_0805_2012Metric_Pad1.15x1.40mm_HandSolder, symbol Device:LED
- added D3, D4: Zener (15V), Package_TO_SOT_SMD:SOT-23, symbol Device:D_Zener
- added J1, J2, J3, J4: Conn_01x03_Pin, Connector_PinHeader_2.54mm:PinHeader_1x03_P2.54mm_Vertical, symbol Connector:Conn_01x03_Pin
- added J5, J6: USB4085-GF-A_REVB, footprints:GCT_USB4085-GF-A_REVB, symbol USB4085-GF-A_REVB:USB4085-GF-A_REVB
- added J7: Conn_01x08_Socket, Connector_Molex:Molex_KK-396_5273-08A_1x08_P3.96mm_Vertical, symbol Connector:Conn_01x08_Socket
- added J8: Conn_01x02_Socket, Connector_AMASS:AMASS_XT60PW-M_1x02_P7.20mm_Horizontal, symbol Connector:Conn_01x02_Socket
- added K1, K2, K3, K4, K5: SRD-05VDC-SL-C, footprints:RELAY_SRD-05VDC-SL-C, symbol SRD-05VDC-SL-C:SRD-05VDC-SL-C
- added Q1, Q2: IRLZ44N, Package_TO_SOT_THT:TO-220-3_Vertical, symbol Transistor_FET:IRLZ44N
- added R10, R11, R12, R13, R2, R3, R5, R7: 10k, Resistor_SMD:R_0805_2012Metric_Pad1.20x1.40mm_HandSolder, symbol Device:R
- added R14: 4, Resistor_SMD:R_0805_2012Metric_Pad1.20x1.40mm_HandSolder, symbol Device:R
- added R15: 4.7k, Resistor_SMD:R_0805_2012Metric_Pad1.20x1.40mm_HandSolder, symbol Device:R
- added R16, R17, R18, R19, R20, R21, R8, R9: 1.1k, Resistor_SMD:R_0805_2012Metric_Pad1.20x1.40mm_HandSolder, symbol Device:R
- added R4, R6: 100, Resistor_SMD:R_0805_2012Metric_Pad1.20x1.40mm_HandSolder, symbol Device:R
- added unit 5 of U2
- added U3: BTS50010-1TAD, Package_TO_SOT_SMD:TO-263-7_TabPin4, symbol Power_Management:BTS50010-1TAD
- added U4, U5: AP22615AWU, Package_TO_SOT_SMD:SOT-23-6, symbol Regulator_Linear:AP22615AWU
- added U6: ULN2002, Package_SO:SOIC-16_3.9x9.9mm_P1.27mm, symbol Transistor_Array:ULN2002
- PS1: footprint PTR08100WVD -> footprints:PTR08100WVD
- R1: footprint (none) -> Resistor_SMD:R_0805_2012Metric_Pad1.20x1.40mm_HandSolder
- U1: footprint RASPBERRY_PI_ZERO_2_W:MODULE_RASPBERRY_PI_ZERO_2_W -> footprints:MODULE_RASPBERRY_PI_ZERO_2_W
- U2: footprint (none) -> Package_SO:SOIC-14_3.9x8.7mm_P1.27mm
Connections:
- net +12V: now also C3.1, D3.1 (K), J8.1 (Pin_1), K1.COM, K2.COM, K3.COM, K4.COM, U3.4 (Vbb)
- net +5V: now also C1.1, C2.1, J1.2 (Pin_2), J2.2 (Pin_2), J3.2 (Pin_2), J4.2 (Pin_2), K1.A1, K2.A1, K3.A1, K4.A1, K5.A1, U2.14 (VCC), U4.6 (IN), U5.6 (IN), U6.9 (COM)
- net GND: now also U2.1, U2.10, U2.13, U2.4, C1.2, C2.2, C3.2, C5.2, D4.1 (K), J1.1 (Pin_1), J2.1 (Pin_1), J3.1 (Pin_1), J4.1 (Pin_1), J5.A1 (GND), J5.A12 (GND), J5.B1 (GND), J5.B12 (GND), J5.S1 (SHELL), J5.S2 (SHELL), J5.S3 (SHELL), J5.S4 (SHELL), J6.A1 (GND), J6.A12 (GND), J6.B1 (GND), J6.B12 (GND), J6.S1 (SHELL), J6.S2 (SHELL), J6.S3 (SHELL), J6.S4 (SHELL), J8.2 (Pin_2), K5.COM, Q1.3 (S), Q2.3 (S), R14.2, R16.2, R17.2, R18.2, R19.2, R2.2, R20.2, R21.2, R3.2, R5.2, R7.2, R8.2, R9.2, U2.7 (GND), U4.2 (GND), U5.2 (GND), U6.8 (GND)
- net FAN_PWM: now reaches U1.12 (GPIO18/GPIO_GEN1)
- net FAN_PWM: now also D5.2 (A), R15.1
- net SERVO_PWM_4: now reaches U1.15 (GPIO22/GPIO_GEN3)
- net SERVO_PWM_4: now also U2.12
- net RASPBERRY_PI_EN: now reaches U1.16 (GPIO23/GPIO_GEN4)
- net RASPBERRY_PI_EN: now also R2.1, U4.4 (EN)
- net HEATED_WINDOW_EN: now reaches U1.18 (GPIO24/GPIO_GEN5)
- net HEATED_WINDOW_EN: now also R4.1
- net EXTRA_LOW_EN: now reaches U1.21 (GPIO9/SPI_MISO)
- net EXTRA_LOW_EN: now also U6.5 (I5)
- net FRONT_FOG_EN: now reaches U1.22 (GPIO25/GPIO_GEN6)
- net FRONT_FOG_EN: now also R6.1
- net EXTRA_HIGH_EN: now reaches U1.24 (GPIO8/SPI_~{CE0})
- net EXTRA_HIGH_EN: now also U6.4 (I4)
- net REAR_FOG_LIGHTS_EN: now reaches U1.26 (GPIO7/SPI_~{CE1})
- net REAR_FOG_LIGHTS_EN: now also U6.3 (I3)
- net INDICATORS_A_EN: now reaches U1.29 (GPIO5)
- net INDICATORS_A_EN: now also U6.1 (I1)
- net INDICATORS_B_EN: now reaches U1.31 (GPIO6)
- net INDICATORS_B_EN: now also U6.2 (I2)
- net SERVO_PWM_1: now reaches U1.35 (GPIO19)
- net SERVO_PWM_1: now also U2.2
- net SERVO_PWM_2: now reaches U1.38 (GPIO20)
- net SERVO_PWM_2: now also U2.5
- net SERVO_PWM_3: now reaches U1.40 (GPIO21)
- net SERVO_PWM_3: now also U2.9
- net at U2.6: now also J2.3 (Pin_3)
- net at U2.11: now also J4.3 (Pin_3)
- net at U2.3: now also J1.3 (Pin_3)
- net at U2.8: now also J3.3 (Pin_3)
- new net: D2.1 (K), R9.1
- new net: D6.1 (K), R17.1
- new net: D6.2 (A), K5.A2, U6.12 (O5)
- new net: D8.1 (K), R19.1
- new net: Q2.1 (G), R6.2, R7.1
- new net: D10.1 (K), R21.1
- new net: D10.2 (A), K1.A2, U6.16 (O1)
- new net: Q1.1 (G), R3.1, R4.2
- new net: D9.1 (K), R20.1
- new net: D7.2 (A), K4.A2, U6.13 (O4)
- new net: D8.2 (A), K3.A2, U6.14 (O3)
- new net: D9.2 (A), K2.A2, U6.15 (O2)
- new net: D7.1 (K), R18.1
- new net: J6.A5 (CC1), R13.2
- new net: J5.A5 (CC1), R10.2
- new net: J5.B5 (CC2), R11.2
- new net: D5.1 (K), R16.1
- new net: C4.1, R15.2, U3.2 (IN)
- new net: J6.B5 (CC2), R12.2
- new net: C4.2, R14.1, U3.1 (GND)
- new net: D3.2 (A), D4.2 (A)
- new net: D1.1 (K), R8.1
- new net DISPLAY_EN: R5.1, U5.4 (EN)
- new net DISPLAY_PWR: D1.2 (A), J6.A4 (VBUS), J6.A9 (VBUS), J6.B4 (VBUS), J6.B9 (VBUS), R12.1, R13.1, U5.1 (OUT)
- new net EXTRA_HIGH: J7.7 (Pin_7), K4.NO
- new net EXTRA_LOW: J7.8 (Pin_8), K5.NO
- new net FAN_OUT: C5.1, J7.1 (Pin_1), U3.5 (OUT), U3.6 (OUT), U3.7 (OUT)
- new net FRONT_FOG_LIGHTS: J7.3 (Pin_3), Q2.2 (D)
- new net HEATED_WINDOW: J7.2 (Pin_2), Q1.2 (D)
- new net INDICATORS_A: J7.4 (Pin_4), K1.NO
- new net INDICATORS_B: J7.5 (Pin_5), K2.NO
- new net RASPBERRY_PI_PWR: D2.2 (A), J5.A4 (VBUS), J5.A9 (VBUS), J5.B4 (VBUS), J5.B9 (VBUS), R10.1, R11.1, U4.1 (OUT)
- new net REAR_FOG_LIGHTS: J7.6 (Pin_6), K3.NO
Other:
- note added: "POWER SWITCHES"
- note added: "SERVO OUTPUTS"
- moved on the sheet: PS1, R1, U1, U2A, U2B, U2C, U2D
